Commit message: Update

File: urdf/mbot.urdf (robot description, URDF)
Before this commit: robot test_robot, 5 links, 4 joints
Links:
- added link aruco_tag; visual mesh filename=aruco_0.obj
- link base_link: geometry collision box size=0.16 0.16 0.12; visual box size=0.18 0.15 0.12
- link left_wheel: geometry collision cylinder length=0.008 radius=0.042; visual cylinder length=0.008 radius=0.042
Joints:
- added joint base_to_aruco_tag: type fixed, parent base_link, child aruco_tag, origin xyz=0 0 0.2 rpy=0 0 0
- joint base_to_front_wheel: origin xyz=0.13 0 0.02 rpy=0 0 0 -> xyz=-0.13 0 0.022 rpy=0 0 0
