Commit message: Both moving in sim

File: urdf/mbot_0.urdf (robot description, URDF)
Before this commit: robot test_robot, 6 links, 5 joints
Links:
- link aruco_tag: geometry visual mesh filename=aruco_0.obj

File: urdf/mbot_1.urdf (robot description, URDF)
Before this commit: robot test_robot, 6 links, 5 joints
Links:
- link aruco_tag: geometry visual mesh filename=aruco_1.obj
